File: pcb/v1/v1.kicad_sch (KiCad schematic)
At the start: 0 parts

Commit message: building pcb
Parts:
- added C1: 100nF, Capacitor_SMD:C_0402_1005Metric, symbol Device:C
- added J1: RPi_GPIO18, Connector_PinHeader_2.54mm:PinHeader_1x02_P2.54mm_Vertical, symbol Connector_Generic:Conn_01x02
- added J2: EXT_5V_IN, Connector_PinHeader_2.54mm:PinHeader_1x02_P2.54mm_Vertical, symbol Connector_Generic:Conn_01x02
- added J3: LED_OUT, Connector_PinHeader_2.54mm:PinHeader_1x03_P2.54mm_Vertical, symbol Connector_Generic:Conn_01x03
- added R1: 10k, Resistor_SMD:R_0402_1005Metric, symbol Device:R
- added R2: 330R, Resistor_SMD:R_0402_1005Metric, symbol Device:R
- added TP1: GPIO_IN, TestPoint:TestPoint_Pad_D1.5mm, symbol Connector:TestPoint
- added TP2: DATA_OUT, TestPoint:TestPoint_Pad_D1.5mm, symbol Connector:TestPoint
- added TP3: 5V, TestPoint:TestPoint_Pad_D1.5mm, symbol Connector:TestPoint
- added TP4: GND, TestPoint:TestPoint_Pad_D1.5mm, symbol Connector:TestPoint
- added U1: SN74AHCT1G125, Package_TO_SOT_SMD:SOT-23-5, symbol 74xGxx:74AHCT1G125
Connections:
- new net: R2.1, U1.4
- new net +5V: C1.1, J2.1 (Pin_1), J3.1 (Pin_1), TP3.1, U1.5 (VCC)
- new net DATA_OUT: J3.2 (Pin_2), R2.2, TP2.1
- new net GND: C1.2, J1.2 (Pin_2), J2.2 (Pin_2), J3.3 (Pin_3), R1.2, TP4.1, U1.1, U1.3 (GND)
- new net GPIO_IN: J1.1 (Pin_1), R1.1, TP1.1, U1.2
Other:
- note added: "*** EXTERNAL 5V (J2) IS NOT CONNECTED TO THE RASPBERRY Pi 5V HEADER ***"
- note added: "J1 carries GPIO18 and GND only. GND is common between the Pi and the external supply - this is the required"
- note added: "J1: 1=GPIO18 2=GND"
- note added: "J2: 1=+5V 2=GND"
- note added: "J3: 1=+5V 2=DATA 3=GND"
- note added: "OE tied low = always enabled"
- note added: "R1 holds GPIO18 low while the Pi is off or the pin is tri-stated. R2 damps ringing - keep close to U1 pin 4. C1 within 3mm of U1 pin 5."
- note added: "SN74AHCT1G125 buffer running at VCC=5V. Its VIH(min) is 2.0V, so 3.3V GPIO logic drives it reliably."
- note added: "WS2812B LEVEL SHIFTER - Raspberry Pi GPIO18 (3.3V) to 5V DATA"
- note added: "signal return path and does not backfeed the Pi. Power this board and the LED strip from the external supply only."
