File: pcb/v1/v1.kicad_pcb (KiCad board)
At the start: 2 copper layers, 60 x 40 mm, 11 parts, among them J1 RPi_GPIO18, J2 EXT_5V_IN, J3 LED_OUT, U1 SN74AHCT1G125

Commit message: Almost done traces
Routing:
- net +5V: track 0.00 -> 114.1 mm
- net /DATA_OUT: track 0.00 -> 28.0 mm
- net /GPIO_IN: track 0.00 -> 25.9 mm
- net GND: track 0.00 -> 13.8 mm
- net Net-(R2-Pad1): track 0.00 -> 1.85 mm
Other:
- board text added: "+5V"
- board text added: "+5V IN"
- board text added: "5V"
- board text added: "DATA"
- board text added: "DATA_OUT"
- board text added: "EXT 5V ONLY - NOT Pi 5V"
- board text added: "GND"
- board text added: "GPIO18"
- board text added: "GPIO_IN"
- board text added: "LED STRIP"
- board text added: "LUMINODE WS2812B LEVEL SHIFTER"
- board text added: "SN74AHCT1G125"
- board text added: "TO RPi"
